File: toolhead/snakeffc-toolhead.kicad_sch (KiCad schematic)
At the start: 13 parts, among them J10 ZMIN, J11 SERVO, J12 E_STEPPER, J13 Conn_01x01, J14 Conn_01x01, J4 Conn_01x26, J5 HEATER_24V, J6 HEATER_SW, J7 THERMISTOR, J8 HOTEND_FAN, J9 PARTCOOLER_FAN, U2 ADXL345

Commit message: toolhead r3 schematic
Parts:
- removed J13, J14: Conn_01x01, Connector_PinHeader_2.54mm:PinHeader_1x01_P2.54mm_Vertical, symbol Connector_Generic:Conn_01x01
- removed J4: Conn_01x26, FFCconnector:FFC26pinTH, symbol Connector_Generic:Conn_01x26
- removed J5: HEATER_24V, Connector_Wire:SolderWire-2.5sqmm_1x01_D2.4mm_OD3.6mm, symbol Connector_Generic:Conn_01x01
- removed J6: HEATER_SW, Connector_Wire:SolderWire-2.5sqmm_1x01_D2.4mm_OD3.6mm, symbol Connector_Generic:Conn_01x01
- removed J7: THERMISTOR, Connector_PinHeader_2.54mm:PinHeader_1x02_P2.54mm_Vertical, symbol Connector_Generic:Conn_01x02
- added J13, J14, J15: X_HOME, Connector_PinHeader_2.54mm:PinHeader_1x02_P2.54mm_Vertical, symbol Connector_Generic:Conn_01x02
- added J4: Conn_01x30, ffc_connectors:ffc-30pin, symbol Connector_Generic:Conn_01x30
- added J5: HEATER, Connector_PinHeader_2.54mm:PinHeader_1x02_P2.54mm_Vertical, symbol Connector_Generic:Conn_01x02
- added J7: THEMISTOR, Connector_PinHeader_2.54mm:PinHeader_1x04_P2.54mm_Vertical, symbol Connector_Generic:Conn_01x04
Connections:
- net +24V: now also J4.1 (Pin_1), J4.2 (Pin_2), J4.3 (Pin_3), J4.4 (Pin_4), J5.1 (Pin_1)
- net +3V3: now also J4.19 (Pin_19)
- net +5V: now also J4.20 (Pin_20), J4.21 (Pin_21)
- net ADXL345_CS: now also J4.22 (Pin_22)
- net ADXL345_SCL: now also J4.18 (Pin_18)
- net ADXL345_SDA: now also J4.24 (Pin_24)
- net ADXL345_SDO: now also J4.23 (Pin_23)
- net GND: now also J13.2 (Pin_2), J14.2 (Pin_2), J15.2 (Pin_2), J4.11 (Pin_11), J4.12 (Pin_12)
- net HEATER_SW: now also J4.27 (Pin_27), J4.28 (Pin_28), J4.29 (Pin_29), J4.30 (Pin_30), J5.2 (Pin_2)
- net HOTEND_FAN_SW: now also J4.25 (Pin_25)
- net PART_FAN_SW: now also J4.26 (Pin_26)
- net STEPPER_A1: now also J4.14 (Pin_14)
- net STEPPER_A2: now also J4.16 (Pin_16)
- net STEPPER_B1: now also J4.15 (Pin_15)
- net STEPPER_B2: now also J4.17 (Pin_17)
- net X_HOME: now also J13.1 (Pin_1), J14.1 (Pin_1), J15.1 (Pin_1), J4.5 (Pin_5)
- net PROBE_ZMIN_BL_WHITE renamed PROBE_ZMIN_24V
- net PROBE_ZMIN_24V: now also J4.10 (Pin_10)
- net SERVO_BL_ORANGE renamed SERVO_NEOPIXEL
- net SERVO_NEOPIXEL: now also J4.13 (Pin_13)
- new net GNDA: J4.6 (Pin_6), J7.1 (Pin_1)
- new net THERM_0: J4.7 (Pin_7), J7.2 (Pin_2)
- new net THERM_AUX_1: J4.8 (Pin_8), J7.3 (Pin_3)
- new net THERM_AUX_2: J4.9 (Pin_9), J7.4 (Pin_4)
Other:
- note added: "SERVO/NEOPIXEL"
- moved on the sheet: C2, J10, J11, J12, J8, J9, U2

Commit message: add footprints
Parts:
- removed J15: X_HOME, Connector_PinHeader_2.54mm:PinHeader_1x02_P2.54mm_Vertical, symbol Connector_Generic:Conn_01x02
- removed J7: THEMISTOR, Connector_PinHeader_2.54mm:PinHeader_1x04_P2.54mm_Vertical, symbol Connector_Generic:Conn_01x04
- added J1: PT100_3PIN, Connector_PinHeader_2.54mm:PinHeader_1x03_P2.54mm_Vertical, symbol Connector_Generic:Conn_01x03
- added J15: AUX1, symbol Connector_Generic:Conn_01x01
- added J16: AUX2, symbol Connector_Generic:Conn_01x01
- added J2: NTC, Connector_PinHeader_2.54mm:PinHeader_1x02_P2.54mm_Vertical, symbol Connector_Generic:Conn_01x02
Connections:
- net GNDA: now also J2.2 (Pin_2)
- net THERM_0: now also J1.1 (Pin_1), J2.1 (Pin_1)
- net THERM_AUX_1: now also J1.2 (Pin_2), J15.1 (Pin_1)
- net THERM_AUX_2: now also J1.3 (Pin_3), J16.1 (Pin_1)
Other:
- moved on the sheet: J8, J9

Commit message: toolhead artwork
Parts:
- removed J1: PT100_3PIN, Connector_PinHeader_2.54mm:PinHeader_1x03_P2.54mm_Vertical, symbol Connector_Generic:Conn_01x03
- removed J15: AUX1, symbol Connector_Generic:Conn_01x01
- removed J2: NTC, Connector_PinHeader_2.54mm:PinHeader_1x02_P2.54mm_Vertical, symbol Connector_Generic:Conn_01x02
- added J1: PT100_NTC, Connector_PinHeader_2.54mm:PinHeader_1x04_P2.54mm_Vertical, symbol Connector_Generic:Conn_01x04
- C2: footprint Capacitor_SMD:C_0805_2012Metric_Pad1.18x1.45mm_HandSolder -> Capacitor_SMD:C_0603_1608Metric
- J13: footprint Connector_PinHeader_2.54mm:PinHeader_1x02_P2.54mm_Vertical -> ffc_connectors:limit_switch
- J16: value AUX2 -> AUX1; footprint (none) -> Connector_PinHeader_2.54mm:PinHeader_1x01_P2.54mm_Vertical
- J5: footprint Connector_PinHeader_2.54mm:PinHeader_1x02_P2.54mm_Vertical -> ffc_connectors:KF301-5.0
Connections:
- net +24V: now also J5.2 (Pin_2); no longer J5.1 (Pin_1)
- net ADXL345_SDA: now also J4.25 (Pin_25); no longer J4.24 (Pin_24)
- net GNDA: now also J4.9 (Pin_9), J1.1 (Pin_1); no longer J4.6 (Pin_6)
- net HEATER_SW: now also J5.1 (Pin_1); no longer J5.2 (Pin_2)
- net HOTEND_FAN_SW: now also J4.24 (Pin_24); no longer J4.25 (Pin_25)
- net THERM_0: now also J4.8 (Pin_8), J1.2 (Pin_2); no longer J4.7 (Pin_7)
- net THERM_AUX_1: now also J16.1 (Pin_1), J4.7 (Pin_7), J1.3 (Pin_3); no longer J4.8 (Pin_8)
- net THERM_AUX_2: now also J4.6 (Pin_6), J1.4 (Pin_4); no longer J16.1 (Pin_1), J4.9 (Pin_9)
Other:
- moved on the sheet: J16

Commit message: r3 jlcpcb
Parts:
- removed J14: X_HOME, Connector_PinHeader_2.54mm:PinHeader_1x02_P2.54mm_Vertical, symbol Connector_Generic:Conn_01x02
Changed lines of the file:
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@@
-    )
-  )
-  (global_label "X_HOME" (shape input) (at 187.96 132.715 180) (fields_autoplaced)
-    (effects (font (size 1.27 1.27)) (justify right))
-    (property "Intersheet References" "${INTERSHEET_REFS}" (id 0) (at 178.1083 132.6356 0)
-      (effects (font (size 1.27 1.27)) (justify right) hide)
     )
   )
@@
     (pin "9")
   )
-  (symbol (lib_id "Connector_Generic:Conn_01x02") (at 193.04 132.715 0) (unit 1)
-    (in_bom yes) (on_board yes) (fields_autoplaced)
-    (property "Reference" "J14" (id 0) (at 196.215 132.7149 0)
-      (effects (font (size 1.27 1.27)) (justify left))
-    )
-    (property "Value" "X_HOME" (id 1) (at 196.215 135.2549 0)
-      (effects (font (size 1.27 1.27)) (justify left))
-    )
-    (property "Footprint" "Connector_PinHeader_2.54mm:PinHeader_1x02_P2.54mm_Vertical" (id 2) (at 193.04 132.715 0)
-      (effects (font (size 1.27 1.27)) hide)
-    )
-    (property "Datasheet" "~" (id 3) (at 193.04 132.715 0)
-      (effects (font (size 1.27 1.27)) hide)
-    )
-    (pin "1")
-    (pin "2")
-  )
   (symbol (lib_id "Connector_Generic:Conn_01x03") (at 193.04 60.325 0) (unit 1)
     (in_bom yes) (on_board yes) (fields_autoplaced)
@@
     )
     (property "Datasheet" "" (id 3) (at 60.325 48.26 0)
-      (effects (font (size 1.27 1.27)) hide)
-    )
-    (pin "1")
-  )
-  (symbol (lib_id "power:GND") (at 187.96 135.255 270) (unit 1)
-    (in_bom yes) (on_board yes) (fields_autoplaced)
-    (property "Reference" "#PWR012" (id 0) (at 181.61 135.255 0)
-      (effects (font (size 1.27 1.27)) hide)
-    )
-    (property "Value" "GND" (id 1) (at 184.15 135.2549 90)
-      (effects (font (size 1.27 1.27)) (justify right))
-    )
-    (property "Footprint" "" (id 2) (at 187.96 135.255 0)
-      (effects (font (size 1.27 1.27)) hide)
-    )
-    (property "Datasheet" "" (id 3) (at 187.96 135.255 0)
       (effects (font (size 1.27 1.27)) hide)
     )
@@
       (reference "#PWR011") (unit 1) (value "GNDA") (footprint "")
     )
-    (path "/f7bbc504-b122-4420-b30b-3fb6f33ff4ef"
-      (reference "#PWR012") (unit 1) (value "GND") (footprint "")
-    )
     (path "/0c31b682-6ce4-4a01-88cd-f78d76f14965"
       (reference "#PWR032") (unit 1) (value "+3.3V") (footprint "")
@@
       (reference "J13") (unit 1) (value "X_HOME") (footprint "ffc_connectors:limit_switch")
     )
-    (path "/a6f80cad-88e6-42b8-bf40-1410708e8221"
-      (reference "J14") (unit 1) (value "X_HOME") (footprint "Connector_PinHeader_2.54mm:PinHeader_1x02_P2.54mm_Vertical")
-    )
     (path "/7632f7c4-2504-4bf4-b023-c0140de6edb1"
